File: PCB/star_watcher/star_watcher.sch (KiCad schematic (older format))
At the start: 44 parts, among them J1 Programming, J2 Motor2, J3 Motor1, J4 input power, J5 UART1, J6 UART2, J7 I2C, U1 ESP32-WROOM-32U, U2 DS3231MZ, U3 MP1584

Commit message: PCB should be feature complete now Just a few capacitors and startup IO stuff missing.
Parts:
- added C10, C11: 10µF, Capacitor_SMD:C_0805_2012Metric, symbol Device:C
- added DS1: HY1602E, Display:HY1602E, symbol Display_Character:HY1602E
- added J8: Micro_SD_Card_Det, Connector_Card:microSD_HC_Hirose_DM3BT-DSF-PEJS, symbol Connector:Micro_SD_Card_Det
- added Q1: Q_PMOS_GDS, Package_TO_SOT_SMD:SOT-23, symbol Device:Q_PMOS_GDS
- added R14: 240, Resistor_SMD:R_0805_2012Metric, symbol Device:R
- added R15: 390, Resistor_SMD:R_0805_2012Metric, symbol Device:R
- added R16: R, Resistor_SMD:R_0805_2012Metric, symbol Device:R
- added R17, R18, R19, R20, R21, R22: 10k, Resistor_SMD:R_0805_2012Metric, symbol Device:R
- added SW1, SW2: Rotary_Encoder_Switch, Button_Switch_THT:KSA_Tactile_SPST, symbol Device:Rotary_Encoder_Switch
- added U4: PCF8574, Package_SO:SOIC-16W_7.5x10.3mm_P1.27mm, symbol Interface_Expansion:PCF8574
- added U5: AMS1117, Package_TO_SOT_SMD:SOT-223, symbol my_components:AMS1117
- R11: value R -> 210k
- R12: value R -> 40.2k
Connections:
- net +3V3: now also C11.2, J8.4 (VDD), R14.2, R17.1, R18.1, R19.1, R20.1, R21.1, R22.1, U4.16 (VDD), U5.2 (Vout), U5.4 (Vout); no longer C4.2, C6.2, C7.2, L1.2
- net DTR: now also SW2.B
- net GND: now also C10.1, C11.1, DS1.3 (VSS), DS1.5 (Vo), DS1.7 (R/~W), J8.11 (SHIELD), J8.6 (VSS), Q1.2 (D), R15.1, SW1.C, SW1.S2, SW2.C, SW2.S2, U4.1 (A0), U4.2 (A1), U4.3 (A2), U4.8 (VSS)
- net RTC_RST: now also U4.11 (P6); no longer U1.27 (IO16)
- net RX2: now also U1.11 (IO26); no longer U1.16 (IO13)
- net SCL: now also U1.37 (IO23), U4.14 (SCL); no longer U1.23 (IO15)
- net SDA: now also U1.36 (IO22), U4.15 (SDA); no longer U1.13 (IO14)
- net TX1: now also U1.10 (IO25); no longer U1.26 (IO4)
- net TX2: now also U1.12 (IO27); no longer U1.14 (IO12)
- net SD_D0: now reaches U1.24 (IO2)
- net SD_D0: now also J8.7 (DAT0), R17.2
- net ROTARY2_PUSH: now reaches U1.5 (SENSOR_VN)
- net ROTARY2_PUSH: now also SW2.S1
- net ROTARY1_B: now reaches U1.6 (IO34)
- net ROTARY1_B: now also SW1.B
- net ROTARY1_PUSH: now reaches U1.7 (IO35)
- net ROTARY1_PUSH: now also SW1.S1
- net LCD_BACKLIGHT: now reaches U1.8 (IO32)
- net LCD_BACKLIGHT: now also Q1.1 (G)
- net ROTARY1_A: now reaches U1.9 (IO33)
- net ROTARY1_A: now also SW1.A
- new net: DS1.1 (LEDK), Q1.3 (S)
- new net: DS1.2 (LEDA), R16.1
- new net: R14.1, R15.2, U5.1 (ADJ)
- new net +5V: C10.2, C4.2, C6.2, C7.2, DS1.4 (VDD), L1.2, R16.2, U5.3 (Vin)
- new net LCD_DB4: DS1.13 (DB4), U4.7 (P3)
- new net LCD_DB5: DS1.14 (DB5), U4.6 (P2)
- new net LCD_DB6: DS1.15 (DB6), U4.5 (P1)
- new net LCD_DB7: DS1.16 (DB7), U4.4 (P0)
- new net LCD_E: DS1.8 (E), U4.10 (P5)
- new net LCD_RS: DS1.6 (RS), U4.9 (P4)
- new net ROTARY2_A: SW2.A, U1.27 (IO16)
- new net SD_CLK: J8.5 (CLK), R21.2, U1.13 (IO14)
- new net SD_CMD: J8.3 (CMD), R22.2, U1.23 (IO15)
- new net SD_D1: J8.8 (DAT1), R18.2, U1.26 (IO4)
- new net SD_D2: J8.1 (DAT2), R20.2, U1.14 (IO12)
- new net SD_D3: J8.2 (DAT3/CD), R19.2, U1.16 (IO13)
- no-connect marks 19 -> 16
Other:
- note added: "TODO: Add elko for drivers"
- note added: "TODO: Pull IO2 low when programming\nRead about the internal LDO selection"
- note removed: "TODO:\n - Display\n - Input Button (rotary encoder?)"
- moved on the sheet: A1, A2, BT1, C1, C2, C3, J1, J2, J3, J5, J6, J7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

Commit message: Use nokia 5110 as display
Parts:
- removed C10, C11: 10µF, Capacitor_SMD:C_0805_2012Metric, symbol Device:C
- removed DS1: HY1602E, Display:HY1602E, symbol Display_Character:HY1602E
- removed Q1: Q_PMOS_GDS, Package_TO_SOT_SMD:SOT-23, symbol Device:Q_PMOS_GDS
- removed R15: 390, Resistor_SMD:R_0805_2012Metric, symbol Device:R
- removed U5: AMS1117, Package_TO_SOT_SMD:SOT-223, symbol my_components:AMS1117
- added Q1: Q_PMOS_DGS, symbol Device:Q_PMOS_DGS
- added R23, R24, R25, R26, R27, R28, R29: 10k, Resistor_SMD:R_0805_2012Metric, symbol Device:R
- added SW3, SW4: SW_Push, symbol Switch:SW_Push
- added U6: 5110, symbol my_components:5110
- R11: value 210k -> R
- R14: value 240 -> R
Connections:
- net LCD_DB4 is gone; now on net ROTARY1_A: U4.7 (P3)
- net LCD_DB5 is gone; now on net ROTARY2_A: U4.6 (P2)
- net LCD_DB6 is gone; now on net ROTARY1_PUSH: U4.5 (P1)
- net LCD_DB7 is gone; now on net ROTARY2_PUSH: U4.4 (P0)
- net LCD_RS is gone; now on net ROTARY1_B: U4.9 (P4)
- net +3V3: now also C4.2, C6.2, C7.2, L1.2, R14.1, Q1.3 (S), R23.2, R24.2, R25.1, R26.1, R27.1, R28.1, R29.1, U6.6 (VCC); no longer R14.2
- net DTR: now also SW4.1; no longer SW2.B
- net GND: now also SW3.2, SW4.2, U6.8 (GND)
- net LCD_BACKLIGHT: now also U1.11 (IO26), Q1.2 (G); no longer U1.8 (IO32)
- net ROTARY1_A: now also R24.1; no longer U1.9 (IO33)
- net ROTARY1_B: now also R26.2; no longer U1.6 (IO34)
- net ROTARY1_PUSH: now also R27.2; no longer U1.7 (IO35)
- net ROTARY2_A: now also R23.1; no longer U1.27 (IO16)
- net ROTARY2_PUSH: now also R28.2; no longer U1.5 (SENSOR_VN)
- net RTC_RST: now also U4.12 (P7); no longer U4.11 (P6)
- net RX1: now also U1.7 (IO35); no longer U1.29 (IO5)
- net RX2: now also U1.6 (IO34); no longer U1.11 (IO26)
- net at R16.1: now also U6.7 (LIGHT)
- removed net +5V: C4.2, C6.2, C7.2, L1.2, R16.2
- net LCD_E renamed ROTARY2_B
- net ROTARY2_B: now also SW2.B, R25.2
- new net: Q1.1 (D), R16.2
- new net CE_5110: U1.27 (IO16), U6.2 (CE)
- new net DC_5110: U1.29 (IO5), U6.3 (DC)
- new net PUSH1: R14.2, SW3.1, U1.5 (SENSOR_VN)
- new net RST_5110: R29.2, U4.11 (P6), U6.1 (RST)
- new net SPI_MOSI: U1.9 (IO33), U6.4 (DIN)
- new net SPI_SCK: U1.8 (IO32), U6.5 (CLK)
- no-connect marks 16 -> 11
Other:
- note added: "If R20 is populated the internal fuse might be required to be set"
- moved on the sheet: R2, R3, SW1, SW2
